Commit message: 添加车臂控制，但是目前有bug，有待改进

File: roboticstoolbox/scripts/mr500_kinova_description/urdf/mr500_kinova.urdf_bk.xacro (robot description, xacro)
@@ -121,10 +121,10 @@
       </collision>
     </link>
-    <joint name="${prefix}joint_1" type="revolute">
+    <joint name="${prefix}joint_1" type="continuous">
       <origin xyz="0 0 0.15643" rpy="-3.1416 0.0 0.0" />
       <parent link="${prefix}base_link" />
       <child link="${prefix}shoulder_link" />
       <axis xyz="0 0 1" />
-      <limit lower="-2.41" upper="2.41" effort="39" velocity="1.3963" />
+      <limit effort="39" velocity="1.3963" />
     </joint>
     <link name="${prefix}bicep_link">
@@ -208,10 +208,10 @@
       </collision>
     </link>
-    <joint name="${prefix}joint_4" type="revolute">
+    <joint name="${prefix}joint_4" type="continuous">
       <origin xyz="0 0.20843 -0.006375" rpy="1.5708 0.0 0.0" />
       <parent link="${prefix}forearm_link" />
       <child link="${prefix}spherical_wrist_1_link" />
       <axis xyz="0 0 1" />
-      <limit lower="-2.66" upper="2.66" effort="39" velocity="1.3963" />
+      <limit effort="9" velocity="1.2218" />
     </joint>
     <link name="${prefix}spherical_wrist_2_link">
@@ -292,10 +292,10 @@
     </link>
     </xacro:unless>
-    <joint name="${prefix}joint_6" type="revolute">
+    <joint name="${prefix}joint_6" type="continuous">
       <origin xyz="0 0.10593 -0.00017505" rpy="1.5708 0.0 0.0" />
       <parent link="${prefix}spherical_wrist_2_link" />
       <child link="${prefix}bracelet_link" />
       <axis xyz="0 0 1" />
-      <limit lower="-2.23" upper="2.23" effort="9" velocity="1.2218" />
+      <limit effort="9" velocity="1.2218" />
     </joint>
     <link name="${prefix}end_effector_link" />
