Commit message: 在多数情况下能够收敛，一些情况下无法收敛

File: roboticstoolbox/scripts/mr500_kinova_description/urdf/mr500_kinova.urdf.xacro (robot description, xacro)
@@ -61,5 +61,5 @@
         <child link="base_link1"/>
         <axis xyz="0 0 1"/>
-        <limit effort="87" lower="-999999" upper="999999" velocity="4.0"/>
+        <limit effort="87" lower="-999999" upper="999999" velocity="1.6"/>
     </joint>
     <joint name="base_joint2"  type="prismatic">
@@ -68,10 +68,10 @@
         <child link="mount_link"/>
         <axis xyz="1 0 0"/>
-        <limit effort="87" lower="-999999" upper="999999" velocity="4.0"/>
+        <limit effort="87" lower="-999999" upper="999999" velocity="1.6"/>
     </joint>
     <joint name="mount_joint" type="fixed">
       <origin
         xyz="0.0 0.0 0.250"
-        rpy="0.0 0.0 0.0"/>
+        rpy="0.0 0.0 3.1416"/>
       <parent link="mount_link"/>
       <child link="kinova_base_link"/>
